File: B0/Reach_B0.brd (EAGLE design)
At the start: 107.3 x 69.5 mm, 238 parts, among them IC1 TMC2130QFN36, IC10 74AHC1G126DCK, IC11 74AHC1G126DCK, IC18 74AHC1G126DCK, IC2 TMC2130QFN36, IC3 74AHC1G126DCK, IC4 74AHC1G126DCK, IC5 74AHC1G126DCK, IC6 74AHC1G126DCK, IC7 74AHC1G126DCK, IC8 TMC2130QFN36, IC9 74AHC1G126DCK, P8 F-2X23-, P9 F-2X23-, Q2 AON6758, Q3 AON6758, U1 SN74AHC595PW, U10 RT8268, U11 PCA9685PW, U18 CAT24C256, U2 SN74AHC595PW, U3 MCP9600, U4 MCP9600, U5 MCP9600, U6 MCP9600, U7 SN74AHC595PW, X1 22-05-7028-02, X11 22-05-7028-02, X14 22-05-7048-04, X2 MSTBA4, X21 MSTBA2, X3 MSTBA2, X4 22-05-7028-02, X5 22-05-7028-02, X6 22-05-7048-04, X7 22-05-7028-02, X8 22-05-7048-04, X9 22-05-7028-02

Commit message: removed LCD jumpers
Parts:
- removed JP4: (no value), SparkFun-PassivesNEW:PAD-JUMPER-2-NC_BY_TRACE_YES_SILK
- removed R88, R89: 0, SparkFun-Resistors:0805
- removed XTC2, XTC3, XTC4: NEWPORT_THERMOCOUPLE_CONNECTORPCC-SMP-V, reach_custom:PCC-SMP-V
- added JP16, JP17, JP18: (no value), SparkFun-ConnectorsNEW:SCREWTERMINAL-5MM-2
- added R61, R62: 330, rcl:R0402
- JP15: device SparkFun-Connectors:SCREWTERMINAL-5MM-2 -> SparkFun-ConnectorsNEW:SCREWTERMINAL-5MM-2
- R66, R67, R77, R78: value 0 -> 330; device SparkFun-Resistors:0805 -> rcl:R0402
- moved R77 62.6 mm to (32.7, 48.8), flipped to the top, turned to 0 degrees
- moved R78 61.1 mm to (33.8, 54.1), flipped to the top, turned to 0 degrees
- moved R67 23.6 mm to (75.0, 62.3), flipped to the top, turned to 0 degrees
- moved R66 23.4 mm to (88.5, 62.2), flipped to the top, turned to 0 degrees
- moved C49 7.63 mm to (93.9, 52.0)
- moved L3 7.63 mm to (98.0, 52.0)
- moved R58 7.63 mm to (95.5, 52.6)
- moved U3 7.63 mm to (90.2, 52.0)
- moved L1 7.63 mm to (96.1, 53.8)
- moved R56 7.63 mm to (95.5, 51.3)
- moved R7 7.63 mm to (89.4, 48.4)
- moved R8 7.63 mm to (87.4, 48.4)
- moved C51 6.25 mm to (79.1, 24.4)
- moved C58 6.25 mm to (85.4, 20.5)
- moved L9 6.25 mm to (89.4, 20.5)
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Connections:
- removed net N$134: R88.2, XTC4.P$1
- removed net N$135: R89.2, XTC4.P$2
- removed net N$900: U7.9
- removed net N$97: R77.2, XTC3.P$1
- removed net N$98: R78.2, XTC3.P$2
- new net N$51: Q3.4, R47.2, R61.1
- new net N$73: Q2.4, R48.2, R62.1
- new net N$83: Q1.1, R19.2, R77.1
- new net N$84: Q6.1, R34.2, R78.1
- net FAN4: now also R78.2; no longer Q6.1, R34.2
- net FAN5: now also R77.2; no longer Q1.1, R19.2
- net FAN6: now also R67.2; no longer Q4.1, R21.2
- net FAN7: now also R66.2; no longer Q5.1, R33.2
- net GND: no longer JP4.1
- net GNDI: no longer JP4.2, R66.1, R67.1, R77.1, R78.1, R88.1, R89.1
- net HEATER_A: now also R61.2; no longer Q3.4, R47.2
- net HEATER_B: now also R62.2; no longer Q2.4, R48.2
- net N$123: now also JP18.2; no longer XTC4.P$4
- net N$130: now also JP18.1; no longer XTC4.P$3
- net N$38: now also JP16.2; no longer XTC2.P$4
- net N$47: now also JP16.1; no longer XTC2.P$3
- net N$76: now also Q5.1, R33.2, R66.1; no longer R66.2, XTC2.P$1
- net N$77: now also Q4.1, R21.2, R67.1; no longer R67.2, XTC2.P$2
- net N$87: now also JP17.2; no longer XTC3.P$4
- net N$92: now also JP17.1; no longer XTC3.P$3
Routing:
- net +3V3: track 330.0 -> 362.1 mm
- net N$133: track 1.37 -> 13.4 mm
- net N$95: track 1.37 -> 13.2 mm
- net N$50: track 1.37 -> 13.1 mm
- net I2C2_SDA: track 39.0 -> 48.5 mm
- net N$72: track 3.71 -> 11.3 mm
- net N$131: track 3.71 -> 9.95 mm
- net N$93: track 3.71 -> 9.82 mm
- net N$48: track 3.71 -> 9.74 mm
- net FAN7: track 62.4 -> 57.1 mm
- net FAN5: track 38.6 -> 33.3 mm
- net FAN4: track 20.4 -> 15.1 mm
- net FAN6: track 50.9 -> 45.6 mm
- net N$11: track 4.67 -> 9.80 mm
- net N$84: track 0.00 -> 4.63 mm
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